File: Esquematicos/CAE32_PCB_V_1.0/CAE32_PCB.kicad_pcb (KiCad board)
At the start: 2 copper layers, 1 part, among them U1 ESP32-S3-WROOM-1

Commit message: Se agregaron archivos .md para dar mas informacion
Parts:
- added U2: 74HC4051, Package_SO:SOIC-16W_5.3x10.2mm_P1.27mm, F.Cu at (85.9, 37.6)
- added U3: 74HC4051, Package_SO:SOIC-16W_5.3x10.2mm_P1.27mm, F.Cu at (86.7, 51.8)
Routing:
- net GNDREF: track 0.00 -> 25.4 mm

Commit message: Actualización del archivo README
Parts:
- added C1: 10uf, Capacitor_SMD:C_0805_2012Metric, F.Cu at (68.6, 37.1)
- added C2: 10uf, Capacitor_SMD:C_0805_2012Metric, F.Cu at (68.6, 34.1)
- added C3: 22uf, Capacitor_SMD:C_0805_2012Metric, F.Cu at (65.0, 47.8)
- added C4: 0.1uf, Capacitor_SMD:C_0805_2012Metric, F.Cu at (69.5, 44.7)
- added C5: 1uf, Capacitor_SMD:C_0805_2012Metric, F.Cu at (65.0, 44.7)
- added C6: 0.1uf, Capacitor_SMD:C_0805_2012Metric, F.Cu at (71.1, 56.4)
- added J1: USB_A, Connector_USB:USB_Micro-B_Wuerth_629105150521, F.Cu at (23.7, 56.6)
- added R1: 10k, Resistor_SMD:R_0805_2012Metric, F.Cu at (69.5, 47.7)
- added R2: 0, Resistor_SMD:R_0805_2012Metric, F.Cu at (80.3, 61.5)
- added U4: SSP1117, Package_TO_SOT_SMD:SOT-223-3_TabPin2, F.Cu at (61.4, 36.7)
- added U5: AD7788BRM, eec:Analog_Devices-AD7788BRM-Level_B, F.Cu at (65.5, 62.0)
Connections:
- U1 pad 1: Net-(U1-Pad1) -> GNDREF
- U1 pad 13: unconnected-(U1-Pad13) -> /D-
- U1 pad 14: unconnected-(U1-Pad14) -> /D+
- U1 pad 2: unconnected-(U1-Pad2) -> +3.3V
- U1 pad 27: unconnected-(U1-Pad27) -> /BOOT
- U1 pad 3: unconnected-(U1-Pad3) -> /EN
- U1 pad 36: unconnected-(U1-Pad36) -> /TX0
- U1 pad 37: unconnected-(U1-Pad37) -> /RX0
- U1 pad 40: Net-(U1-Pad1) -> GNDREF
- U1 pad 41: Net-(U1-Pad1) -> GNDREF
- U2 pad 8: GNDREF -> unconnected-(U2-Pad8)
Other:
- copper layers 2 -> 4
