File: Esquematicos/CAE32_PCB_V_1.0/dfg.kicad_sch (KiCad schematic)
At the start: 1 part, among them U3 74HC4051

Commit message: Actualización del archivo README
Parts:
- U3: Campo4 (none) -> ffff
Changed lines of the file:
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@@
+      (effects (font (size 1.27 1.27)) hide)
+    )
+    (property "Campo4" "ffff" (id 4) (at 195.58 74.93 0)
       (effects (font (size 1.27 1.27)) hide)
     )
