File: Esquematicos/CAE32_PCB_V_0.2/Modular/Modular/Modular.kicad_sch (KiCad schematic)
At the start: 21 parts, among them J1 Steering Wheel Feedback, J2 Pedals, J3 Shifter, J4 Accessory_2, J5 Accessory_1, J6 Conn_01x04, J7 Screw_Terminal_01x02, P1 USB_C_Plug_USB2.0, U1 ESP32-S3-WROOM-1, U3 LDL1117

Commit message: Diseño de Pcb y Boom, de placa de pedales 1.0V
Parts:
- added D1, D2: UDD32, CAE:UDD32, symbol CAE32:UDD32
Connections:
- net +5V: now also J1.7, J2.7, J3.7, J4.7, J5.7; no longer J1.2, J2.2, J3.2, J4.2, J5.2
- net D+: now also D1.1
- net D-: now also D2.1
- net GNDREF: now also D1.2, D2.2
- net MOSI: now also J1.2, J2.2, J3.2, J4.2, J5.2; no longer J1.3, J2.3, J3.3, J4.3, J5.3
- net SCLK: now also J1.8, J2.8, J3.8, J4.8, J5.8; no longer J1.5, J2.5, J3.5, J4.5, J5.5
Other:
- note added: "5v supply"
- note added: "Accessories modules"
- moved on the sheet: F1, J7

Commit message: Actualización de README
Parts:
- added D3: LED, LED_SMD:LED_0805_2012Metric_Pad1.15x1.40mm_HandSolder, symbol Device:LED
- renumbered C7 to C1, C8 to C2, C5 to C3, C6 to C4, C2 to C5, C4 to C6, J6 to J1, J7 to J2, J5 to J3, J1 to J4, J2 to J5, J3 to J6, J4 to J7, U3 to U2
Connections:
- net +3.3V: now also D3.2 (A)
- net CS_PDL: now also U1.18 (GPIO10/TOUCH10/ADC1_CH9/FSPICS0/FSPIIO4/SUBSPICS0); no longer U1.17 (GPIO9/TOUCH9/ADC1_CH8/FSPIHD/SUBSPIHD)
- net CS_SWF: now also U1.17 (GPIO9/TOUCH9/ADC1_CH8/FSPIHD/SUBSPIHD); no longer U1.18 (GPIO10/TOUCH10/ADC1_CH9/FSPICS0/FSPIIO4/SUBSPICS0)
- net GNDREF: now also D3.1 (K)
Other:
- note added: "Power Indicator"

Commit message: Actualización de Gerbers e indicador de status de conexión
Parts:
- removed P1: USB_C_Plug_USB2.0, Connector_USB:USB_C_Receptacle_Palconn_UTC16-G, symbol Connector:USB_C_Plug_USB2.0
- added D4: D_Schottky, Diode_SMD:D_SMA_Handsoldering, symbol Device:D_Schottky
- added J1: USB_OTG, Connector_USB:USB_Micro-B_Amphenol_10104110_Horizontal, symbol Connector:USB_OTG
- renumbered J1 to J2, J2 to J3, J3 to J4, J4 to J5, J5 to J6, J6 to J7, J7 to J8
Connections:
- net D+: now also D2.1, J1.3 (D+); no longer D1.1
- net D-: now also D1.1, J1.2 (D-); no longer D2.1
- net GNDREF: now also D4.2 (A), J1.4 (ID), J1.5 (GND), J1.6 (Shield)
- net at F1.1, J3.2 (Pin_2): now also D4.1 (K)
- no-connect marks 0 -> 1
Other:
- note added: "Usb connection"
- note removed: "Fuse Invert polarity protection"
- moved on the sheet: D1, D2, F1
