File: Esquematicos/CAE32_PCB_V_0.2/Pedals/Pedals/Pedals.kicad_sch (KiCad schematic)
At the start: 16 parts, among them U1 STM32G070RBT6, U2 LDL1117

Commit message: Correciones de errores PCB:pedales y hall
Parts:
- added ID1, ID2, ID3: LED, LED_SMD:LED_0805_2012Metric_Pad1.15x1.40mm_HandSolder, symbol Device:LED
- added MODE1: SW_Push, Button_Switch_SMD:SW_Push_1P1T_NO_6x6mm_H9.5mm, symbol Switch:SW_Push
- added R2, R3, R4: 10, Resistor_SMD:R_0805_2012Metric_Pad1.20x1.40mm_HandSolder, symbol Device:R_Small_US
- added R5: 43, Resistor_SMD:R_0805_2012Metric_Pad1.20x1.40mm_HandSolder, symbol Device:R_Small_US
- added UART_PGRM1: Conn_01x05_Female, Connector_PinHeader_2.54mm:PinHeader_1x05_P2.54mm_Vertical, symbol Connector:Conn_01x05_Female
Connections:
- net +3.3V: now also R5.1, UART_PGRM1.4 (Pin_4); no longer PWD1.2 (A)
- net GNDREF: now also ID1.1 (K), ID2.1 (K), ID3.1 (K), MODE1.2, UART_PGRM1.1 (Pin_1)
- net MISO: no longer U1.10 (PA3)
- net MOSI: now also U1.23 (PA12_[PA10]); no longer U1.21 (PA10), U1.9 (PA2)
- net SCKL: no longer U1.7 (PA0)
- net IND0: now reaches U1.30 (PB6)
- net IND0: now also R2.1
- net IND1: now reaches U1.31 (PB7)
- net IND1: now also R3.1
- net IND2: now reaches U1.32 (PB8)
- net IND2: now also R4.1
- net CS_PROGRAM: no longer names the net of DATA1.5
- net CS_PROGRAM: no longer U1.1 (PB9)
- new net: ID3.2 (A), R4.2
- new net: ID2.2 (A), R3.2
- new net: PWD1.2 (A), R5.2
- new net: ID1.2 (A), R2.2
- new net MODE: MODE1.1, U1.1 (PB9)
- new net USART_RX: U1.10 (PA3), UART_PGRM1.3 (Pin_3)
- new net USART_TX: U1.9 (PA2), UART_PGRM1.2 (Pin_2)
- no-connect marks 0 -> 1
Other:
- note added: "Activate Update Mode"
- note added: "MISC Indicators"
- note added: "UART PGRM"

Commit message: Ultima revision de PCBs
Parts:
- added 5V1, GND1: TestPoint, TestPoint:TestPoint_Pad_D3.0mm, symbol Connector:TestPoint
Connections:
- net +5V: now also 5V1.1
- net GNDREF: now also GND1.1
Other:
- note added: "Power source 5v"
- company: (none) -> Techtep
- title: (none) -> CAE32 pedals
- moved on the sheet: BOOT1, C1, C2, C3, ID1, ID2, ID3, R1, R2, R3, R4, RST1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
